Commit message: added lidar dependencies and structure

File: linorobot2_description/urdf/minidrone_properties.urdf.xacro (robot description, xacro)
@@ -18,3 +18,6 @@
     <origin xyz="0.55 0 0.16" rpy="0 0 0"/>
   </xacro:property>
+  <xacro:property name="lidar_pose">
+    <origin xyz="0.0 0 0.16" rpy="0 0 0"/>
+  </xacro:property>
 </robot>

File: linorobot2_description/urdf/robots/minidrone.urdf.xacro (robot description, xacro)
@@ -9,4 +9,5 @@
   <xacro:include filename="$(find linorobot2_description)/urdf/sensors/gps.urdf.xacro" />
   <xacro:include filename="$(find linorobot2_description)/urdf/controllers/skid_steer.urdf.xacro" />
+  <xacro:include filename="$(find velodyne_description)/urdf/VLP-16.urdf.xacro" />
   <xacro:base
     length="${base_length}"
@@ -55,7 +56,9 @@
   <xacro:imu />
   <xacro:gps />
-  <xacro:generic_laser>
-    <xacro:insert_block name="laser_pose" />
-  </xacro:generic_laser>
+  <!--
+  <xacro:VLP-16>
+    <xacro:insert_block name="lidar_pose" />
+  </xacro:VLP-16>
+  -->
   <xacro:stereo_camera>
     <xacro:insert_block name="stereo_camera_pose" />

Commit message: repositioned camera

File: linorobot2_description/urdf/minidrone_properties.urdf.xacro (robot description, xacro)
@@ -16,5 +16,5 @@
   </xacro:property>
   <xacro:property name="stereo_camera_pose">
-    <origin xyz="0.55 0 0.16" rpy="0 0 0"/>
+    <origin xyz="0.4 0 0.45" rpy="0 0.5 0"/>
   </xacro:property>
   <xacro:property name="lidar_pose">
