Commit message: added steering joints

File: linorobot2_description/urdf/controllers/ackermann_drive.urdf.xacro (robot description, xacro)
@@ -11,6 +11,6 @@
         <rear_left_joint>rear_left_wheel_joint</rear_left_joint>
         <rear_right_joint>rear_right_wheel_joint</rear_right_joint>
-        <left_steering_joint>front_left_wheel_joint</left_steering_joint>
-        <right_steering_joint>front_right_wheel_joint</right_steering_joint>
+        <left_steering_joint>front_left_steering_joint</left_steering_joint>
+        <right_steering_joint>front_right_steering_joint</right_steering_joint>
         <wheel_separation>${wheel_separation}</wheel_separation>
         <wheel_diameter>${wheel_radius * 2}</wheel_diameter>

File: linorobot2_description/urdf/mech/wheel.urdf.xacro (robot description, xacro)
@@ -2,4 +2,5 @@
 <robot xmlns:xacro="http://ros.org/wiki/xacro">
   <xacro:macro name="wheel" params="side radius width pos_x pos_y pos_z mass">
+    <link name="${side}_steering_link"/>
     <link name="${side}_wheel_link">
       <visual>
@@ -36,9 +37,15 @@
       </visual>
     </gazebo>
+    <joint name="${side}_steering_joint" type="continuous">
+      <axis xyz="0 0 1"/>
+      <parent link="base_link"/>
+      <child link="${side}_wheel_steering_link"/>
+      <origin xyz="${x_pos} ${y_pos} ${z_pos}" rpy="0 0 0"/>
+    </joint>
     <joint name="${side}_wheel_joint" type="continuous">
       <axis xyz="0 1 0" />
-      <parent link="base_link"/>
+      <parent link="${side}_steering_link"/>
       <child link="${side}_wheel_link"/>
-      <origin xyz="${pos_x} ${pos_y} ${pos_z}" rpy="0 0 0"/>
+      <origin xyz="0 0 0" rpy="0 0 0"/>
     </joint>
   </xacro:macro>
